File: MidPlate/Manta60_Mid_Left.kicad_pcb (KiCad board)
At the start: 2 copper layers, 168.9 x 121.4 mm, 103 parts, among them P1 LED-pin, SW1 SW_Push, SW10 SW_Push, SW11 SW_Push, SW12 SW_Push, SW13 SW_Push, SW14 SW_Push, SW15 SW_Push, SW16 SW_Push, SW17 SW_Push, SW18 SW_Push, SW19 SW_Push, SW2 SW_Push, SW20 SW_Push, SW21 SW_Push, SW22 SW_Push, SW23 SW_Push, SW24 SW_Push, SW25 SW_Push, SW26 SW_Push, SW27 SW_Push, SW28 SW_Push, SW29 SW_Push, SW3 SW_Push, SW30 SW_Push, SW31 SW_Push, SW32 SW_Push, SW34 SW_Push, SW35 SW_Push, SW4 SW_Push, SW5 SW_Push, SW6 SW_Push, SW7 SW_Push, SW8 SW_Push, SW9 SW_Push, T1 TRRS, U1 ProMicro

Commit message: update
Parts:
- removed JP8: SolderJumper, library:Jumper3
- added ?: C_0805, Capacitors_SMD:C_0805_HandSoldering, F.Cu at (174.0, 82.3)
- added ?: , library:GND, F.Cu at (84.6, 123.6)
- added J1: BAT, manta60:PH_2Pin_Top, F.Cu at (176.8, 82.3)
- added JP1: , library:Jumper3, B.Cu at (190.0, 74.5)
- added JP2: , library:Jumper3, B.Cu at (187.2, 74.5)
- added JP3: , library:Jumper3, B.Cu at (184.4, 74.6)
- added JP4: , library:Jumper3, B.Cu at (181.6, 74.6)
- added SW33: SW_Push, manta60:CherryMX_Hotswap_left, F.Cu at (179.4, 144.4)
- JP5, JP6, JP7: value SolderJumper -> (none)
- O1: footprint library:OLED -> manta60:OLED
- SW1, SW10, SW11, SW12, SW13, SW14, SW15, SW16, SW17, SW18, SW19, SW2, SW20, SW21, SW22, SW23, SW24, SW25, SW26, SW27, SW28, SW29 (x2), SW3, SW30, SW31, SW32, SW35, SW4, SW5 (x2), SW6, SW7, SW8, SW9: footprint manta60:Kailh-socket -> manta60:CherryMX_Hotswap_left
- U1: footprint library:ProMicro -> manta60:ProMicro
- moved JP5 9.71 mm to (188.1, 81.8)
- moved JP7 8.31 mm to (191.2, 81.8)
- moved JP6 7.26 mm to (184.9, 81.8)
- moved P1 4.00 mm to (193.7, 104.1)
- moved REF** 4.00 mm to (197.5, 101.5)
- moved REF** 4.00 mm to (197.5, 106.6)
- moved REF** 4.00 mm to (197.5, 104.1)
- moved S1 4.00 mm to (188.7, 104.1)
- moved D29 3.81 mm to (176.4, 113.0)
- moved D33 3.81 mm to (180.2, 113.2)
- moved H12 0.24 mm to (193.8, 75.6)
- renumbered H1 to ?
Connections:
- JP5 pad 1: Net-(JP4-Pad1) -> Net-(JP5-Pad1)
- JP5 pad 2: SDA -> SCL
- JP6 pad 1: Net-(JP3-Pad1) -> Net-(JP6-Pad1)
- JP6 pad 2: SCL -> SDA
- JP7 pad 1: Net-(JP2-Pad1) -> Net-(JP5-Pad1)
- JP7 pad 2: VCC -> Data
- T1 pad B: Net-(T1-PadB) -> Net-(JP6-Pad1)
- T1 pad C: Data -> Net-(JP5-Pad1)
Routing:
- net BAT_GND: track 0.00 -> 69.3 mm
- net BAT: track 0.00 -> 48.1 mm
- net GND: track 23.3 -> 49.3 mm, vias 33 -> 42
- net Col4: track 229.8 -> 204.0 mm
- net Col5: track 215.9 -> 191.3 mm, vias 3 -> 5
- net Col0: track 297.5 -> 274.9 mm
- net Col2: track 252.9 -> 231.0 mm
- net Col3: track 232.1 -> 211.0 mm
- net Col1: track 239.2 -> 218.2 mm
- net Col6: track 203.1 -> 185.8 mm
- net SCL: track 28.6 -> 39.1 mm
- net SDA: track 28.9 -> 38.3 mm
- net Net-(JP6-Pad1): track 0.00 -> 8.51 mm, vias 0 -> 1
- net Net-(JP5-Pad1): track 0.00 -> 7.67 mm
- net Data: track 44.6 -> 37.6 mm, vias 0 -> 1
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Other:
- outline, holes or cut-outs redrawn
- board text added: "+"
- board text added: "-"
- board text added: "BAT"
- board text added: "C0"
- board text added: "C6"
- board text added: "Col0"
- board text added: "Col1"
- board text added: "Col2"
- board text added: "Col3"
- board text added: "Col4"
- board text added: "Col5"
- board text added: "Col6"
- board text added: "I2C"
- board text added: "LED"
- board text added: "OLED"
- board text added: "R0"
- board text added: "R4"
- board text added: "RX"
- board text added: "Row0"
- board text added: "Row1"
- board text added: "Row2"
- board text added: "Row3"
- board text added: "Row4"
